File: HARDWARE/EDA/KICAD/IVD/IVD.kicad_pcb (KiCad board)
At the start: 2 copper layers, 62 x 24 mm, 16 parts, among them J1 V_INPUT, J2 Digital_Info, Q1 BC549, U1 4N25

Commit message: adjust PCB
Parts:
- moved D3 15.6 mm to (126.0, 81.0), turned to 0 degrees
- moved RV1 15.0 mm to (110.0, 80.0)
- moved D5 13.0 mm to (123.0, 88.0), turned to 180 degrees
- moved D1 10.8 mm to (123.0, 79.0), turned to 180 degrees
- moved J2 10.1 mm to (151.0, 73.0)
- moved Q1 8.12 mm to (142.0, 80.0), turned to 90 degrees
- moved R1 8.07 mm to (133.6, 88.1), turned to 180 degrees
- moved D4 6.00 mm to (113.0, 85.0), turned to 0 degrees
- moved C1 4.34 mm to (134.0, 78.0), turned to 90 degrees
- moved D2 4.24 mm to (113.0, 82.0), turned to 0 degrees
- moved R2 3.69 mm to (133.6, 85.0), turned to 180 degrees
- moved R3 3.30 mm to (147.1, 78.0)
- moved R4 2.19 mm to (148.0, 73.0), turned to 180 degrees
Routing:
- net Net-(C1-Pad2): track 54.7 -> 34.0 mm
- net Net-(D4-Pad1): track 26.7 -> 13.7 mm
- net Net-(C1-Pad1): track 32.1 -> 19.8 mm
- net GNDD: track 14.5 -> 3.00 mm
- net +5VD: track 27.0 -> 17.1 mm
- net Net-(D1-Pad1): track 24.6 -> 16.8 mm
- net Net-(Q1-Pad2): track 11.6 -> 5.32 mm
- net V_Signal: track 17.6 -> 11.8 mm
- net Net-(D1-Pad2): track 15.6 -> 17.6 mm

Commit message: finished board
Parts:
- added D6: LED, LED_THT:LED_D5.0mm, F.Cu at (151.0, 85.0)
- added D7: LED, LED_THT:LED_D5.0mm_IRGrey, F.Cu at (154.0, 73.0)
- added R5: 100R, Resistor_THT:R_Axial_DIN0207_L6.3mm_D2.5mm_P7.62mm_Horizontal, F.Cu at (150.0, 73.0)
- added R6: 100R, Resistor_THT:R_Axial_DIN0207_L6.3mm_D2.5mm_P7.62mm_Horizontal, F.Cu at (154.0, 78.0)
- moved J2 11.7 mm to (157.0, 83.0)
Routing:
- net GNDD: track 3.00 -> 18.4 mm
- net V_Signal: track 11.8 -> 24.8 mm
- net +5VD: track 17.1 -> 27.9 mm
- net Net-(D6-Pad1): track 0.00 -> 4.79 mm
- net Net-(D7-Pad2): track 0.00 -> 2.46 mm
- net Net-(R3-Pad2): track 3.92 -> 4.67 mm
Other:
- board size 62 x 24 mm -> 64 x 21 mm
