File: HARDWARE/EDA/KICAD/IVD/IVD.sch (KiCad schematic (older format))
At the start: 16 parts, among them J1 V_INPUT, J2 Digital_Info, Q1 BC549, U1 4N25

Commit message: PCB finished
Parts:
- C1: value CP -> 3V; footprint (none) -> Capacitor_THT:CP_Radial_D10.0mm_P3.50mm
Changed lines of the file:
@@
 P 3150 1550
 F 0 "C1" H 3268 1596 50  0000 L CNN
-F 1 "CP" H 3268 1505 50  0000 L CNN
-F 2 "" H 3188 1400 50  0001 C CNN
+F 1 "3V" H 3268 1505 50  0000 L CNN
+F 2 "Capacitor_THT:CP_Radial_D10.0mm_P3.50mm" H 3188 1400 50  0001 C CNN
 F 3 "~" H 3150 1550 50  0001 C CNN
 	1    3150 1550

Commit message: finished board
Parts:
- added D6: LED, LED_THT:LED_D5.0mm, symbol Device:LED
- added D7: LED, LED_THT:LED_D5.0mm_IRGrey, symbol Device:LED
- added R5, R6: 100R, Resistor_THT:R_Axial_DIN0207_L6.3mm_D2.5mm_P7.62mm_Horizontal, symbol Device:R
Connections:
- net +5VD: now also D6.2 (A)
- net GNDD: now also D7.1 (K), R5.1
- net V_Signal: now also R6.2
- new net: D6.1 (K), R5.2
- new net: D7.2 (A), R6.1
Changed lines of the file:
@@
 Wire Wire Line
 	6400 1800 6500 1800
+$Comp
+L power:+5VD #PWR06
+U 1 1 6178A8A6
+P 7450 1250
+F 0 "#PWR06" H 7450 1100 50  0001 C CNN
+F 1 "+5VD" H 7465 1423 50  0000 C CNN
+F 2 "" H 7450 1250 50  0001 C CNN
+F 3 "" H 7450 1250 50  0001 C CNN
+	1    7450 1250
+	1    0    0    -1
+$EndComp
+$Comp
+L power:GNDD #PWR07
+U 1 1 6178AC16
+P 7450 2000
+F 0 "#PWR07" H 7450 1750 50  0001 C CNN
+F 1 "GNDD" H 7454 1845 50  0000 C CNN
+F 2 "" H 7450 2000 50  0001 C CNN
+F 3 "" H 7450 2000 50  0001 C CNN
+	1    7450 2000
+	1    0    0    -1
+$EndComp
+$Comp
+L Device:LED D6
+U 1 1 6178B5DE
+P 7450 1450
+F 0 "D6" V 7489 1333 50  0000 R CNN
+F 1 "LED" V 7398 1333 50  0000 R CNN
+F 2 "LED_THT:LED_D5.0mm" H 7450 1450 50  0001 C CNN
+F 3 "~" H 7450 1450 50  0001 C CNN
+	1    7450 1450
+	0    -1   -1   0
+$EndComp
+$Comp
+L Device:R R5
+U 1 1 617932DD
+P 7450 1800
+F 0 "R5" V 7243 1800 50  0000 C CNN
+F 1 "100R" V 7334 1800 50  0000 C CNN
+F 2 "Resistor_THT:R_Axial_DIN0207_L6.3mm_D2.5mm_P7.62mm_Horizontal" V 7380 1800 50  0001 C CNN
+F 3 "~" H 7450 1800 50  0001 C CNN
+	1    7450 1800
+	-1   0    0    1
+$EndComp
+Wire Wire Line
+	7450 1600 7450 1650
+Wire Wire Line
+	7450 1300 7450 1250
+Wire Wire Line
+	7450 1950 7450 2000
+$Comp
+L power:GNDD #PWR08
+U 1 1 6179E0C0
+P 7950 2000
+F 0 "#PWR08" H 7950 1750 50  0001 C CNN
+F 1 "GNDD" H 7954 1845 50  0000 C CNN
+F 2 "" H 7950 2000 50  0001 C CNN
+F 3 "" H 7950 2000 50  0001 C CNN
+	1    7950 2000
+	1    0    0    -1
+$EndComp
+$Comp
+L Device:LED D7
+U 1 1 6179E0C6
+P 7950 1800
+F 0 "D7" V 7989 1683 50  0000 R CNN
+F 1 "LED" V 7898 1683 50  0000 R CNN
+F 2 "LED_THT:LED_D5.0mm_IRGrey" H 7950 1800 50  0001 C CNN
+F 3 "~" H 7950 1800 50  0001 C CNN
+	1    7950 1800
+	0    -1   -1   0
+$EndComp
+$Comp
+L Device:R R6
+U 1 1 6179E0CC
+P 7950 1450
+F 0 "R6" V 7743 1450 50  0000 C CNN
+F 1 "100R" V 7834 1450 50  0000 C CNN
+F 2 "Resistor_THT:R_Axial_DIN0207_L6.3mm_D2.5mm_P7.62mm_Horizontal" V 7880 1450 50  0001 C CNN
+F 3 "~" H 7950 1450 50  0001 C CNN
+	1    7950 1450
+	-1   0    0    1
+$EndComp
+Wire Wire Line
+	7950 1600 7950 1650
+Wire Wire Line
+	7950 1300 7950 1250
+Wire Wire Line
+	7950 1950 7950 2000
+Text GLabel 7950 1250 1    50   Input ~ 0
+V_Signal
 $EndSCHEMATC
